File: hardware/NES_Controller_Breakout.kicad_pcb (KiCad board)
At the start: 2 copper layers, 50 x 50 mm, 6 parts, among them J2 Conn_01x05_Socket

Commit message: Routed PCB
Parts:
- removed REF** (x4): MountingHole_2.7mm_M2.5_DIN965_Pad, MountingHole:MountingHole_2.7mm_M2.5_DIN965_Pad
- added H1: MountingHole_Pad, MountingHole:MountingHole_2.7mm_M2.5_Pad, F.Cu at (176.9, 100.0)
- added H2: MountingHole_Pad, MountingHole:MountingHole_2.7mm_M2.5_Pad, F.Cu at (136.9, 100.0)
- added H3: MountingHole_Pad, MountingHole:MountingHole_2.7mm_M2.5_Pad, F.Cu at (176.9, 140.0)
- added H4: MountingHole_Pad, MountingHole:MountingHole_2.7mm_M2.5_Pad, F.Cu at (136.9, 140.0)
Routing:
- net VCC: track 0.00 -> 23.6 mm
- net Data: track 0.00 -> 20.8 mm
- net Load: track 0.00 -> 20.1 mm
- net Clock: track 0.00 -> 19.5 mm
- added copper zone on B.Cu, net GND
- added copper zone on F.Cu, net GND
