File: hardware/NES_Controller_Breakout.kicad_sch (KiCad schematic)
At the start: 2 parts, among them J2 Conn_01x05_Socket

Commit message: Routed PCB
Parts:
- added H1, H2, H3, H4: MountingHole_Pad, MountingHole:MountingHole_2.7mm_M2.5_Pad, symbol Mechanical:MountingHole_Pad
Connections:
- net GND: now also H1.1, H2.1, H3.1, H4.1
