File: hardware/NES_Controller_Breakout_Board.kicad_pcb (KiCad board)
At the start: 2 copper layers, 50 x 50 mm, 6 parts, among them J2 Conn_01x05_Socket

Commit message: Finished design
Other:
- board text added: "JLCJLCJLCJLC"
